Commit message: Mapping done

File: udacity_bot/urdf/udacity_bot.xacro (robot description, xacro)
@@ -160,4 +160,14 @@
         <parent link="chassis"/>
     </joint>
+    <link name="camera_link_optical">
+    </link>
+    <joint name="camera_optical_joint" type="fixed">
+        <!-- these values have to be these values otherwise the gazebo camera
+        image won't be aligned properly with the frame it is supposedly
+        originating from -->
+        <origin xyz="0 0 0" rpy="${-pi/2} 0 ${-pi/2}"/>
+        <parent link="camera"/>
+        <child link="camera_link_optical"/>
+      </joint>
     <link name='hokuyo'>
         <inertial>
